File: HagiwoDualVCARev2_Panel.kicad_pcb (KiCad board)
At the start: 2 copper layers, 40.3 x 128.5 mm, 14 parts

Commit message: ready for production
Parts:
- removed the REF** at (81.3, 95.3)
- removed the REF** at (81.3, 162.6)
- removed the REF** at (81.3, 152.4)
- removed the REF** at (60.9, 162.6)
- removed the REF** at (61.0, 152.4)
- removed the REF** at (61.0, 142.2)
- removed the REF** at (61.0, 68.6)
- removed the REF** at (81.3, 121.9)
- removed the REF** at (81.3, 142.2)
- removed the REF** at (61.0, 121.9)
- removed the REF** at (81.3, 68.6)
- removed the REF** at (61.0, 95.3)
- added REF**: Faceplate_Hole_Pot_9mm, PCM_4ms_Faceplate:Faceplate_Hole_Pot_9mm, F.Cu at (81.3, 68.6)
- added REF**: GND, PCM_4ms_Faceplate:Faceplate_Hole_Jack_3.5mm, F.Cu at (61.0, 152.4)
- added REF**: Faceplate_Hole_Pot_9mm, PCM_4ms_Faceplate:Faceplate_Hole_Pot_9mm, F.Cu at (61.0, 121.9)
- added REF**: GND, PCM_4ms_Faceplate:Faceplate_Hole_Jack_3.5mm, F.Cu at (81.3, 152.4)
- added REF**: Faceplate_Hole_Pot_9mm, PCM_4ms_Faceplate:Faceplate_Hole_Pot_9mm, F.Cu at (81.3, 121.9)
- added REF**: GND, PCM_4ms_Faceplate:Faceplate_Hole_Jack_3.5mm, F.Cu at (81.3, 142.2)
- added REF**: GND, PCM_4ms_Faceplate:Faceplate_Hole_Jack_3.5mm, F.Cu at (81.3, 162.6)
- added REF**: GND, PCM_4ms_Faceplate:Faceplate_Hole_Jack_3.5mm, F.Cu at (61.0, 142.2)
- added REF**: GND, PCM_4ms_Faceplate:Faceplate_Hole_Jack_3.5mm, F.Cu at (60.9, 162.6)
- added REF**: Faceplate_Hole_Pot_9mm, PCM_4ms_Faceplate:Faceplate_Hole_Pot_9mm, F.Cu at (81.3, 95.3)
- added REF**: Faceplate_Hole_Pot_9mm, PCM_4ms_Faceplate:Faceplate_Hole_Pot_9mm, F.Cu at (61.0, 68.6)
- added REF**: Faceplate_Hole_Pot_9mm, PCM_4ms_Faceplate:Faceplate_Hole_Pot_9mm, F.Cu at (61.0, 95.3)
